File: avrusb.kicad_pcb (KiCad board)
At the start: 2 copper layers, 50 x 41 mm, 26 parts, among them CON1 AVR-ISP-6, J1 Conn_01x03, J2 USB_OTG, J3 Conn_01x04, J4 Conn_01x22, SW1 SW_Push, U1 AT90USB162-16AU, Y1 16 MHz

Commit message: Added github url
Other:
- board text added: "https://github.com/RobertZ2011 /at90usbbasic.git"
Changed lines of the file:
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@@
     (area 93.949999 88.949999 144.050001 130.050001)
     (thickness 1.6)
-    (drawings 26)
+    (drawings 27)
     (tracks 404)
     (zones 0)
@@
   )
   (setup
-    (last_trace_width 0.4)
+    (last_trace_width 0.25)
     (user_trace_width 0.4)
     (trace_clearance 0.2)
@@
       (xy -0.017575 -3.712307) (xy 0 -3.712308) (xy 0.139878 -3.712224)) (layer F.SilkS) (width 0.01))
   )
+  (gr_text "https://github.com/RobertZ2011\n/at90usbbasic.git" (at 115 101) (layer B.SilkS)
+    (effects (font (size 0.5 0.5) (thickness 0.125)) (justify left mirror))
+  )
   (gr_text "Version 1.0.0" (at 108 99) (layer B.SilkS)
